File: MainBoard/MainBoard.kicad_pcb (KiCad board)
At the start: 4 copper layers, 100 x 100 mm, 141 parts, among them J1 12VIN, J2 CTRL, J3 Conn_JTAG, J4 USB_Mini, J5 FPGA_JTAG, J6 Conn_02x07, J7 Conn_02x20, J8 Conn_02x20, J9 Conn_02x07, U1 LXDC55F, U10 LV8548MC, U11 LV8548MC, U12 LV8548MC, U13 LV8548MC, U14 LV8548MC, U15 LV8548MC, U16 LV8548MC, U17 LV8548MC, U18 TBD62083, U19 74VHC540, U2 RX71M_144LQFP_Sonar, U20 74VHC540, U21 74VHC540, U22 LV8548MC, U23 LV8548MC, U24 LV8548MC, U25 LV8548MC, U26 LV8548MC, U27 LV8548MC, U28 LV8548MC, U29 LV8548MC, U3 AS4C32M16SA-7TCN, U30 LV8548MC, U4 MAX10_10M16SC_Sonar, U5 74VHC540, U6 74VHC540, U7 74VHC540, U8 LV8548MC, U9 LV8548MC

Commit message: メインボード完成
Parts:
- added J10: MountingHole, Mounting_Holes:MountingHole_3.2mm_M3_Pad, F.Cu at (40.0, 55.0)
- added J11: MountingHole, Mounting_Holes:MountingHole_3.2mm_M3_Pad, F.Cu at (130.0, 55.0)
- added J12: MountingHole, Mounting_Holes:MountingHole_3.2mm_M3_Pad, F.Cu at (130.0, 145.0)
- added J13: MountingHole, Mounting_Holes:MountingHole_3.2mm_M3_Pad, F.Cu at (40.0, 145.0)
- moved C44 31.1 mm to (64.2, 103.5)
- moved R21 2.66 mm to (70.0, 112.8), turned to 180 degrees
- moved R19 1.00 mm to (95.0, 133.0)
- moved C6 0.75 mm to (108.5, 122.5)
- moved C12 0.50 mm to (82.2, 121.8)
- moved C13 0.50 mm to (82.2, 126.8)
- moved C41 0.40 mm to (85.0, 71.6)
- moved C10 0.25 mm to (88.2, 106.5)
- moved C29 0.25 mm to (78.0, 98.0)
- moved C9 0.25 mm to (94.2, 106.5)
- turned C17 to 180 degrees
- turned C21 to 90 degrees
Routing:
- net GND: track 0.00 -> 1217.6 mm, vias 0 -> 219
- net +3V3: track 0.00 -> 294.2 mm, vias 0 -> 57
- net +12V: track 0.00 -> 79.9 mm, vias 0 -> 19
- net /MCU_UB: track 0.00 -> 72.9 mm, vias 0 -> 1
- net /MIC7: track 0.00 -> 67.0 mm
- net /MIC6: track 0.00 -> 65.5 mm
- net /MICCLK_B: track 0.00 -> 64.4 mm, vias 0 -> 1
- net /MIC9: track 0.00 -> 62.2 mm, vias 0 -> 1
- net SP37: track 0.00 -> 61.9 mm, vias 0 -> 3
- net /MIC11: track 0.00 -> 60.5 mm, vias 0 -> 1
- net /MIC8: track 0.00 -> 60.5 mm, vias 0 -> 1
- net SP36: track 0.00 -> 59.0 mm, vias 0 -> 3
- net /MIC10: track 0.00 -> 58.0 mm, vias 0 -> 1
- net /HSYNC: track 0.00 -> 57.4 mm, vias 0 -> 2
- net /PIXD6: track 0.00 -> 57.2 mm, vias 0 -> 2
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- added copper zone on In1.Cu, net +12V
- added copper zone on In1.Cu, net +3V3
- added copper zone on B.Cu, net GND
- added copper zone on F.Cu, net GND
- added copper zone on In1.Cu, net GND
- added copper zone on In2.Cu, net GND
Other:
- net class Default: clearance 0.21 -> 0.2
- rule trace_clearance: 0.21 -> 0.2
- board text added: "12V IN"
- board text added: "CTRL I/F"
- board text added: "Designed by TamapochiOne"
- board text added: "FPGA JTAG"
- board text added: "MCU JTAG"
- board text added: "Sonar / MainBoard"
- board text added: "USB"
