File: MainBoard/MainBoard.sch (KiCad schematic (older format))
At the start: 87 parts, among them J1 12VIN, J2 CTRL, J3 Conn_JTAG, J4 USB_Mini, J5 FPGA_JTAG, J6 Conn_02x07, J7 Conn_02x20, J8 Conn_02x20, J9 Conn_02x07, U1 LXDC55F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

Commit message: メインボード完成
Parts:
- added J10, J11, J12, J13: MountingHole, Mounting_Holes:MountingHole_3.2mm_M3_Pad, symbol Conn_01x01
Connections:
- net GND: now also J10.1 (Pin_1), J11.1 (Pin_1), J12.1 (Pin_1), J13.1 (Pin_1)
Other:
- note added: "FPGA\n0.1u x 23"
- note removed: "FPGA\n0.1u x 24"
- moved on the sheet: C44
Changed lines of the file:
@@
 Connection ~ 9500 9850
 Wire Wire Line
-	11100 10100 11100 10150
+	11100 10150 11100 10100
 Wire Wire Line
 	9300 10150 11500 10150
@@
 	9300 10800 9300 10900
 Wire Wire Line
-	9300 10550 11500 10550
+	9300 10550 11300 10550
 Wire Wire Line
 	11100 10550 11100 10600
@@
 Connection ~ 9500 10550
 Wire Wire Line
-	11100 10800 11100 10850
-Wire Wire Line
-	9300 10850 11500 10850
+	11100 10850 11100 10800
+Wire Wire Line
+	9300 10850 11300 10850
 Connection ~ 9300 10850
 Wire Wire Line
@@
 L C_Small C44
 U 1 1 5A24277F
-P 11500 10700
-F 0 "C44" H 11510 10770 50  0000 L CNN
-F 1 "0.1u" H 11510 10620 50  0001 L CNN
-F 2 "Capacitors_SMD:C_0402" H 11500 10700 50  0001 C CNN
-F 3 "" H 11500 10700 50  0001 C CNN
-	1    11500 10700
+P 3750 9900
+F 0 "C44" H 3600 9800 50  0000 L CNN
+F 1 "0.1u" H 3760 9820 50  0001 L CNN
+F 2 "Capacitors_SMD:C_0402" H 3750 9900 50  0001 C CNN
+F 3 "" H 3750 9900 50  0001 C CNN
+	1    3750 9900
 	1    0    0    -1
 $EndComp
@@
 	11300 10100 11300 10150
 Connection ~ 11300 10150
-Wire Wire Line
-	11500 10550 11500 10600
 Connection ~ 11100 10550
 Wire Wire Line
-	11300 10600 11300 10550
-Connection ~ 11300 10550
-Wire Wire Line
-	11500 10850 11500 10800
+	11300 10550 11300 10600
 Connection ~ 11100 10850
 Wire Wire Line
-	11300 10800 11300 10850
-Connection ~ 11300 10850
+	11300 10850 11300 10800
 Text Notes 10200 10450 0    60   ~ 0
-FPGA\n0.1u x 24
+FPGA\n0.1u x 23
 $Comp
 L C_Small C14
@@
 Connection ~ 7550 6700
 Wire Wire Line
-	8750 6750 8750 6700
+	8750 6700 8750 6750
 Wire Wire Line
 	8550 6750 8550 6700
@@
 Connection ~ 7550 7000
 Wire Wire Line
-	8750 6950 8750 7000
+	8750 7000 8750 6950
 Wire Wire Line
 	8550 6950 8550 7000
@@
 SDRAM\n0.1u x 7
 Wire Wire Line
-	8750 7000 7550 7000
-Wire Wire Line
-	8750 6700 7550 6700
+	7550 7000 8750 7000
+Wire Wire Line
+	7550 6700 8750 6700
 $Comp
 L C_Small C3
@@
 Connection ~ 5750 8250
 Wire Wire Line
-	5950 8300 5950 8250
+	5950 8250 5950 8300
 Connection ~ 5950 8250
 Connection ~ 5750 8550
 Wire Wire Line
-	5950 8500 5950 8550
+	5950 8550 5950 8500
 Connection ~ 5950 8550
 Text Notes 4800 8150 0    60   ~ 0
 MCU\n0.1u x 11
 Wire Wire Line
-	5950 8250 3950 8250
-Wire Wire Line
-	5950 8550 3950 8550
+	3950 8250 5950 8250
+Wire Wire Line
+	3950 8550 5950 8550
 $Comp
 L +12V #PWR050
@@
 	1450 950  1450 1100
 Connection ~ 1450 1100
+Wire Wire Line
+	3950 9800 3750 9800
+Wire Wire Line
+	3950 10000 3750 10000
+Connection ~ 3950 10000
+Connection ~ 3950 9800
+$Comp
+L Conn_01x01 J10
+U 1 1 5A2FAC00
+P 6900 9700
+F 0 "J10" H 6900 9800 50  0000 C CNN
+F 1 "MountingHole" H 6900 9600 50  0000 C CNN
+F 2 "Mounting_Holes:MountingHole_3.2mm_M3_Pad" H 6900 9700 50  0001 C CNN
+F 3 "" H 6900 9700 50  0001 C CNN
+	1    6900 9700
+	1    0    0    -1
+$EndComp
+$Comp
+L Conn_01x01 J11
+U 1 1 5A2FAFCA
+P 6900 10000
+F 0 "J11" H 6900 10100 50  0000 C CNN
+F 1 "MountingHole" H 6900 9900 50  0000 C CNN
+F 2 "Mounting_Holes:MountingHole_3.2mm_M3_Pad" H 6900 10000 50  0001 C CNN
+F 3 "" H 6900 10000 50  0001 C CNN
+	1    6900 10000
+	1    0    0    -1
+$EndComp
+$Comp
+L Conn_01x01 J12
+U 1 1 5A2FB0F1
+P 6900 10300
+F 0 "J12" H 6900 10400 50  0000 C CNN
+F 1 "MountingHole" H 6900 10200 50  0000 C CNN
+F 2 "Mounting_Holes:MountingHole_3.2mm_M3_Pad" H 6900 10300 50  0001 C CNN
+F 3 "" H 6900 10300 50  0001 C CNN
+	1    6900 10300
+	1    0    0    -1
+$EndComp
+$Comp
+L Conn_01x01 J13
+U 1 1 5A2FB219
+P 6900 10600
+F 0 "J13" H 6900 10700 50  0000 C CNN
+F 1 "MountingHole" H 6900 10500 50  0000 C CNN
+F 2 "Mounting_Holes:MountingHole_3.2mm_M3_Pad" H 6900 10600 50  0001 C CNN
+F 3 "" H 6900 10600 50  0001 C CNN
+	1    6900 10600
+	1    0    0    -1
+$EndComp
+$Comp
+L GND #PWR051
+U 1 1 5A2FB72B
+P 6600 10800
+F 0 "#PWR051" H 6600 10550 50  0001 C CNN
+F 1 "GND" H 6600 10650 50  0001 C CNN
+F 2 "" H 6600 10800 50  0001 C CNN
+F 3 "" H 6600 10800 50  0001 C CNN
+	1    6600 10800
+	1    0    0    -1
+$EndComp
+Wire Wire Line
+	6700 9700 6600 9700
+Wire Wire Line
+	6600 9700 6600 10800
+Wire Wire Line
+	6700 10000 6600 10000
+Connection ~ 6600 10000
+Wire Wire Line
+	6700 10300 6600 10300
+Connection ~ 6600 10300
+Wire Wire Line
+	6600 10600 6700 10600
+Connection ~ 6600 10600
 $EndSCHEMATC
